File: hw/rpi-hat/rpi.sch (EAGLE design)
At the start: 30 parts, among them U1 BSS138, U2 BSS138, U3 BSS138

Commit message: hw/rpi-ha: add bleeder resistors for external LEDs
Parts:
- added R14, R15: 1k, rcl:R-EU_R0805
- R10, R12: value 150R -> 200R
- R2: value 10k -> 1k
Connections:
- net N$3: now also R14.2
- net N$6: now also R14.1
- net N$7: now also R15.2
- net N$8: now also R15.1
Changed lines of the file:
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@@
 <part name="X1" library="con-wago-500" library_urn="urn:adsk.eagle:library:195" deviceset="W237-102" device="" package3d_urn="urn:adsk.eagle:package:10688/1"/>
 <part name="U$2" library="parts" deviceset="JW2SN-DC12V" device=""/>
-<part name="R2" library="rcl" library_urn="urn:adsk.eagle:library:334" deviceset="R-EU_" device="R0805" package3d_urn="urn:adsk.eagle:package:23553/2" value="10k"/>
+<part name="R2" library="rcl" library_urn="urn:adsk.eagle:library:334" deviceset="R-EU_" device="R0805" package3d_urn="urn:adsk.eagle:package:23553/2" value="1k"/>
 <part name="GND1" library="supply1" library_urn="urn:adsk.eagle:library:371" deviceset="GND" device=""/>
 <part name="P+1" library="supply1" library_urn="urn:adsk.eagle:library:371" deviceset="+12V" device=""/>
@@
 <part name="U2" library="parts" deviceset="BSS138" device=""/>
 <part name="LED1" library="pinhead" library_urn="urn:adsk.eagle:library:325" deviceset="PINHD-1X2" device="" package3d_urn="urn:adsk.eagle:package:22435/2"/>
-<part name="R10" library="rcl" library_urn="urn:adsk.eagle:library:334" deviceset="R-EU_" device="R0805" package3d_urn="urn:adsk.eagle:package:23553/2" value="150R"/>
+<part name="R10" library="rcl" library_urn="urn:adsk.eagle:library:334" deviceset="R-EU_" device="R0805" package3d_urn="urn:adsk.eagle:package:23553/2" value="200R"/>
 <part name="P+10" library="supply1" library_urn="urn:adsk.eagle:library:371" deviceset="+5V" device=""/>
 <part name="R11" library="rcl" library_urn="urn:adsk.eagle:library:334" deviceset="R-EU_" device="R0805" package3d_urn="urn:adsk.eagle:package:23553/2" value="10k"/>
@@
 <part name="U3" library="parts" deviceset="BSS138" device=""/>
 <part name="LED2" library="pinhead" library_urn="urn:adsk.eagle:library:325" deviceset="PINHD-1X2" device="" package3d_urn="urn:adsk.eagle:package:22435/2"/>
-<part name="R12" library="rcl" library_urn="urn:adsk.eagle:library:334" deviceset="R-EU_" device="R0805" package3d_urn="urn:adsk.eagle:package:23553/2" value="150R"/>
+<part name="R12" library="rcl" library_urn="urn:adsk.eagle:library:334" deviceset="R-EU_" device="R0805" package3d_urn="urn:adsk.eagle:package:23553/2" value="200R"/>
 <part name="P+11" library="supply1" library_urn="urn:adsk.eagle:library:371" deviceset="+5V" device=""/>
+<part name="R14" library="rcl" library_urn="urn:adsk.eagle:library:334" deviceset="R-EU_" device="R0805" package3d_urn="urn:adsk.eagle:package:23553/2" value="1k"/>
+<part name="R15" library="rcl" library_urn="urn:adsk.eagle:library:334" deviceset="R-EU_" device="R0805" package3d_urn="urn:adsk.eagle:package:23553/2" value="1k"/>
 </parts>
 <sheets>
@@
 <instance part="P+11" gate="1" x="-63.5" y="88.9" smashed="yes">
 <attribute name="VALUE" x="-66.04" y="83.82" size="1.778" layer="96" rot="R90"/>
+</instance>
+<instance part="R14" gate="G$1" x="-48.26" y="142.24" smashed="yes" rot="R270">
+<attribute name="NAME" x="-46.7614" y="146.05" size="1.778" layer="95" rot="R270"/>
+<attribute name="VALUE" x="-51.562" y="146.05" size="1.778" layer="96" rot="R270"/>
+</instance>
+<instance part="R15" gate="G$1" x="-50.8" y="68.58" smashed="yes" rot="R270">
+<attribute name="NAME" x="-49.3014" y="72.39" size="1.778" layer="95" rot="R270"/>
+<attribute name="VALUE" x="-54.102" y="72.39" size="1.778" layer="96" rot="R270"/>
 </instance>
 </instances>
@@
 <pinref part="LED1" gate="G$1" pin="2"/>
 <wire x1="-58.42" y1="139.7" x2="-63.5" y2="139.7" width="0.1524" layer="91"/>
-<wire x1="-63.5" y1="139.7" x2="-63.5" y2="132.08" width="0.1524" layer="91"/>
+<wire x1="-63.5" y1="139.7" x2="-63.5" y2="134.62" width="0.1524" layer="91"/>
+<pinref part="R14" gate="G$1" pin="2"/>
+<wire x1="-63.5" y1="134.62" x2="-63.5" y2="132.08" width="0.1524" layer="91"/>
+<wire x1="-63.5" y1="134.62" x2="-48.26" y2="134.62" width="0.1524" layer="91"/>
+<wire x1="-48.26" y1="134.62" x2="-48.26" y2="137.16" width="0.1524" layer="91"/>
+<junction x="-63.5" y="134.62"/>
 </segment>
 </net>
@@
 <wire x1="-58.42" y1="142.24" x2="-63.5" y2="142.24" width="0.1524" layer="91"/>
 <wire x1="-63.5" y1="142.24" x2="-63.5" y2="147.32" width="0.1524" layer="91"/>
+<pinref part="R14" gate="G$1" pin="1"/>
+<wire x1="-48.26" y1="147.32" x2="-63.5" y2="147.32" width="0.1524" layer="91"/>
+<junction x="-63.5" y="147.32"/>
 </segment>
 </net>
@@
 <pinref part="LED2" gate="G$1" pin="2"/>
 <wire x1="-58.42" y1="66.04" x2="-63.5" y2="66.04" width="0.1524" layer="91"/>
-<wire x1="-63.5" y1="66.04" x2="-63.5" y2="58.42" width="0.1524" layer="91"/>
+<wire x1="-63.5" y1="66.04" x2="-63.5" y2="60.96" width="0.1524" layer="91"/>
+<pinref part="R15" gate="G$1" pin="2"/>
+<wire x1="-63.5" y1="60.96" x2="-63.5" y2="58.42" width="0.1524" layer="91"/>
+<wire x1="-50.8" y1="63.5" x2="-50.8" y2="60.96" width="0.1524" layer="91"/>
+<wire x1="-50.8" y1="60.96" x2="-63.5" y2="60.96" width="0.1524" layer="91"/>
+<junction x="-63.5" y="60.96"/>
 </segment>
 </net>
@@
 <wire x1="-58.42" y1="68.58" x2="-63.5" y2="68.58" width="0.1524" layer="91"/>
 <wire x1="-63.5" y1="68.58" x2="-63.5" y2="73.66" width="0.1524" layer="91"/>
-</segment>
-</net>
+<pinref part="R15" gate="G$1" pin="1"/>
+<wire x1="-63.5" y1="73.66" x2="-50.8" y2="73.66" width="0.1524" layer="91"/>
+<junction x="-63.5" y="73.66"/>
+</segment>
+</net>
